Commit message: polishing simulation

File: franka_description/molds/polishing_mold.xacro (robot description, xacro)
@@ -9,4 +9,5 @@
       </visual>
       <collision>
+        <origin xyz="0 0 0" rpy="${-pi/2} 0 0"/>
         <geometry>
           <mesh filename="package://franka_description/meshes/visual/polishing_mold.dae"/>

File: franka_description/polishing_simulation/polishing_tool.xacro (robot description, xacro)
@@ -21,9 +21,16 @@
       </collision>
       <inertial>
-        <origin xyz="0.0460 -0.0460 0.1150" rpy="-0.7856 1.0472 0"/>
+        <origin xyz="0 0 0" rpy="0 0 0"/>
         <mass value="0.610"/>
         <inertia ixx="0.1" ixy="0.0" ixz="0.0" iyy="0.1" iyz="0.0" izz="0.1"/>
       </inertial>
     </link>
+    <link name="${ns}_EE"/>
+    <joint name="${ns}_EE_joint" type="fixed">
+      <origin xyz="0.0460 -0.0460 0.1150" rpy="0 1.0472 -0.7854"/>
+      <parent link="${ns}_link8"/>
+      <child link="${ns}_EE"/>
+      <axis xyz="0 0 0"/>
+    </joint>
   </xacro:macro>
 </robot>

File: franka_description/simulation/hand.xacro (robot description, xacro)
@@ -77,4 +77,11 @@
       <mimic joint="${ns}_finger_joint1" />
     </joint>
+    <link name="${ns}_EE"/>
+    <joint name="${ns}_EE_joint" type="fixed">
+      <origin xyz="0 0 0.1034" rpy="0 0 -0.7854"/>
+      <parent link="${ns}_link8"/>
+      <child link="${ns}_EE"/>
+      <axis xyz="0 0 0"/>
+    </joint>
   </xacro:macro>
 </robot>

Commit message: Adding polishing_mold to franka_simulation package

File: franka_description/molds/polishing_mold.xacro (robot description, xacro)
@@ -1,17 +1,33 @@
 <?xml version="1.0" encoding="utf-8"?>
 <robot xmlns:xacro="http://www.ros.org/wiki/xacro" name="polishing_mold">
-    <link name="polishing_mold">
-      <visual>
-        <origin xyz="0 0 0" rpy="${-pi/2} 0 0"/>
-        <geometry>
-          <mesh filename="package://franka_description/meshes/visual/polishing_mold.dae"/>
-        </geometry>
-      </visual>
-      <collision>
-        <origin xyz="0 0 0" rpy="${-pi/2} 0 0"/>
-        <geometry>
-          <mesh filename="package://franka_description/meshes/visual/polishing_mold.dae"/>
-        </geometry>
-      </collision>
-    </link>
+  <!-- Import all Gazebo-customization elements, including Gazebo colors -->
+  <xacro:include filename="$(find franka_description)/molds/polishing_mold.gazebo" />
+  <!-- Used for fixing mold to Gazebo 'base_link' -->
+  <link name="world"/>
+  <joint name="mold_to_world" type="fixed">
+    <parent link="world"/>
+    <child link="polishing_mold"/>
+    <origin xyz="0.471134 -0.422512 0.091579" rpy="0.0 0.0 0.0" />
+    <dynamics damping="1.0" friction="0.0"/>
+  </joint>
+  <!-- polishing_mold Link -->
+  <link name="polishing_mold">
+    <visual>
+      <origin xyz="0.0 0.0 0.0" rpy="${-pi/2} 0.0 0.0"/>
+      <geometry>
+        <mesh filename="package://franka_description/meshes/visual/polishing_mold.dae"/>
+      </geometry>
+    </visual>
+    <collision>
+      <origin xyz="0.0 0.0 0.0" rpy="${-pi/2} 0.0 0.0"/>
+      <geometry>
+        <mesh filename="package://franka_description/meshes/visual/polishing_mold.dae"/>
+      </geometry>
+    </collision>
+    <inertial>
+      <origin xyz="0.0 0.0 0.0" rpy="0.0 0.0 0.0"/>
+      <mass value="10"/>
+      <inertia ixx="1.0" ixy="0.0" ixz="0.0" iyy="1.0" iyz="0.0" izz="1.0"/>
+    </inertial>
+  </link>
 </robot>

Commit message: update franka_simulation package

File: franka_description/molds/polishing_mold.xacro (robot description, xacro)
@@ -27,6 +27,6 @@
     <inertial>
       <origin xyz="0.0 0.0 0.0" rpy="0.0 0.0 0.0"/>
-      <mass value="10"/>
-      <inertia ixx="1.0" ixy="0.0" ixz="0.0" iyy="1.0" iyz="0.0" izz="1.0"/>
+      <mass value="50"/>
+      <inertia ixx="5.0" ixy="0.0" ixz="0.0" iyy="5.0" iyz="0.0" izz="5.0"/>
     </inertial>
   </link>

Commit message: meshes update

File: franka_description/molds/polishing_mold.xacro (robot description, xacro)
@@ -14,5 +14,5 @@
   <link name="polishing_mold">
     <visual>
-      <origin xyz="0.0 0.0 0.0" rpy="${-pi/2} 0.0 0.0"/>
+      <origin xyz="0.0 0.0 0.0" rpy="0.0 0.0 0.0"/>
       <geometry>
         <mesh filename="package://franka_description/meshes/visual/polishing_mold.dae"/>
@@ -20,7 +20,7 @@
     </visual>
     <collision>
-      <origin xyz="0.0 0.0 0.0" rpy="${-pi/2} 0.0 0.0"/>
+      <origin xyz="0.0 0.0 0.0" rpy="0.0 0.0 0.0"/>
       <geometry>
-        <mesh filename="package://franka_description/meshes/visual/polishing_mold.dae"/>
+        <mesh filename="package://franka_description/meshes/collision/polishing_mold.stl"/>
       </geometry>
     </collision>

File: franka_description/polishing_simulation/panda_arm_polishing_tool.urdf.xacro (robot description, xacro)
@@ -7,5 +7,5 @@
   <xacro:include filename="$(find franka_description)/polishing_simulation/panda.transmission.xacro"/>
   <xacro:panda_arm />
-  <xacro:polishing_tool ns="panda" rpy="${-pi} 0 ${-pi/4 + pi}" connected_to="panda_link8"/>
+  <xacro:polishing_tool ns="panda" rpy="0 0 ${-pi/4}" connected_to="panda_link8"/>
   <xacro:panda_gazebo robot_name="$(arg robot_name)" />
   <xacro:panda_transmission robot_name="$(arg robot_name)"/>

File: franka_description/polishing_simulation/polishing_tool.xacro (robot description, xacro)
@@ -17,5 +17,5 @@
       <collision>
         <geometry>
-          <mesh filename="package://franka_description/meshes/visual/polishing_tool.dae"/>
+          <mesh filename="package://franka_description/meshes/collision/polishing_tool.stl"/>
         </geometry>
       </collision>

File: franka_description/robots/panda_arm_polishing_tool.urdf.xacro (robot description, xacro)
@@ -4,4 +4,4 @@
   <xacro:include filename="$(find franka_description)/robots/polishing_tool.xacro"/>
   <xacro:panda_arm />
-  <xacro:polishing_tool ns="panda" rpy="${-pi} 0 ${-pi/4 + pi}" connected_to="panda_link8"/>
+  <xacro:polishing_tool ns="panda" rpy="0 0 ${-pi/4}" connected_to="panda_link8"/>
 </robot>

File: franka_description/robots/polishing_tool.xacro (robot description, xacro)
@@ -17,5 +17,5 @@
       <collision>
         <geometry>
-          <mesh filename="package://franka_description/meshes/visual/polishing_tool.dae"/>
+          <mesh filename="package://franka_description/meshes/collision/polishing_tool.stl"/>
         </geometry>
       </collision>
