Commit message: polishing tool update

File: franka_description/polishing_simulation/molds/polishing_mold.xacro (robot description, xacro)
@@ -2,5 +2,5 @@
 <robot xmlns:xacro="http://www.ros.org/wiki/xacro" name="polishing_mold">
   <!-- Import all Gazebo-customization elements, including Gazebo colors -->
-  <xacro:include filename="$(find franka_description)/molds/polishing_mold.gazebo" />
+  <xacro:include filename="$(find franka_description)/polishing_simulation/molds/polishing_mold.gazebo" />
   <!-- Used for fixing mold to Gazebo 'base_link' -->
   <link name="world"/>

File: franka_description/polishing_simulation/polishing_tool.xacro (robot description, xacro)
@@ -23,10 +23,10 @@
         <origin xyz="0 0 0" rpy="0 0 0"/>
         <mass value="0.610"/>
-        <inertia ixx="0.1" ixy="0.0" ixz="0.0" iyy="0.1" iyz="0.0" izz="0.1"/>
+        <inertia ixx="0.000883318125" ixy="0.0" ixz="0.0" iyy="0.000883318125" iyz="0.0" izz="0.00030263625"/>
       </inertial>
     </link>
     <link name="${ns}_EE"/>
     <joint name="${ns}_EE_joint" type="fixed">
-      <origin xyz="0.0460 -0.0460 0.1150" rpy="0 1.0472 -0.7854"/>
+      <origin xyz="0.0403 -0.0403 0.1200" rpy="0 1.0472 -0.7854"/>
       <parent link="${ns}_link8"/>
       <child link="${ns}_EE"/>

Commit message: polishing controller optimization

File: franka_description/polishing_simulation/molds/polishing_mold.xacro (robot description, xacro)
@@ -8,5 +8,5 @@
     <parent link="world"/>
     <child link="polishing_mold"/>
-    <origin xyz="0.471134 -0.422512 0.091579" rpy="0.0 0.0 0.0" />
+    <origin xyz="0.465994 -0.408933 0.0877107" rpy="0.0 0.0 0.0" />
     <dynamics damping="1.0" friction="0.0"/>
   </joint>

Commit message: simulation optimizations

File: franka_description/polishing_simulation/molds/polishing_mold.xacro (robot description, xacro)
@@ -28,5 +28,5 @@
       <origin xyz="0.0 0.0 0.0" rpy="0.0 0.0 0.0"/>
       <mass value="50"/>
-      <inertia ixx="5.0" ixy="0.0" ixz="0.0" iyy="5.0" iyz="0.0" izz="5.0"/>
+      <inertia ixx="1.0" ixy="0.0" ixz="0.0" iyy="1.0" iyz="0.0" izz="1.0"/>
     </inertial>
   </link>
